File: flightController_Local_Main/flightController.kicad_sch (KiCad schematic)
At the start: 53 parts, among them J1 U.FL-R-SMT10, J2 Conn_ARM_SWD, J3 USBC, U1 BD33IA5WEFJ-E2, U11 LIS2MDLTR, U2 TESEO-LIV3F, U3 DPS368XTSA1, U4 STM32H723VETx, U5 TPS22944DCKR, U6 TPS562201DDCR, U7 MIC2004-0.5YM5-TR, U8 LM66100DCKR, U9 LM66100DCKR

Commit message: Adding all step files and footprints
Parts:
- added C24, C34: 10nF, Capacitor_SMD:C_0603_1608Metric, symbol Device:C_Small
- added C27, C33: 0.1uF, Capacitor_SMD:C_0603_1608Metric, symbol Device:C_Small
- added C28: 0.8pF, Capacitor_SMD:C_0603_1608Metric, symbol Device:C_Small
- added C29, C30: 1.2pF, Capacitor_SMD:C_0603_1608Metric, symbol Device:C_Small
- added C31: 0.5pF, Capacitor_SMD:C_0603_1608Metric, symbol Device:C_Small
- added C32: 100pF, Capacitor_SMD:C_0603_1608Metric, symbol Device:C_Small
- added C35: 470nF, Capacitor_SMD:C_0603_1608Metric, symbol Device:C_Small
- added C36, C37: 22uF, Capacitor_SMD:C_0805_2012Metric, symbol Device:C
- added C38, C39: 10uF, Capacitor_SMD:C_1206_3216Metric, symbol Device:C
- added C40, C41: 0.1uF, Capacitor_SMD:C_0603_1608Metric, symbol Device:C
- added C42: 10uF, Capacitor_SMD:C_0805_2012Metric, symbol Device:C
- added J4: U.FL-R-SMT10, Library:U.FL_CONN_v.UL, symbol U.FL_CONN_v.UL:U.FL-R-SMT10
- added J5: XT60-M, Library:XT60-M, symbol XT60-M:XT60-M
- added L3: 3.0nH, Library:3.0nH_Inductor, symbol Device:L_Small
- added L4: 2.5nH, Library:3.0nH_Inductor, symbol Device:L_Small
- added L5: 15uH, Library:15uH_Inductor, symbol Device:L_Small
- added L6: 4.7uH, Library:4.7uH_7.18A, symbol Device:L
- added M1, M2: Motor_Servo, Connector_JST:JST_XH_B3B-XH-AM_1x03_P2.50mm_Vertical, symbol Motor:Motor_Servo
- added R10: 0, Resistor_SMD:R_0603_1608Metric, symbol Device:R_Small_US
- added R11, R12: 10k, Resistor_SMD:R_0603_1608Metric, symbol Device:R_US
- added R13: 68.1k, Resistor_SMD:R_0603_1608Metric, symbol Device:R_US
- added U10: SX1281IMLTRT, Library:XCVR_SX1281IMLTRT, symbol SX1281IMLTRT:SX1281IMLTRT
- added U12: TPS562201DDCR, Library:3.3Buck, symbol 3.3Buck:TPS562201DDCR
- added XTAL1: NX2016SA-52MHZ-EXS00A-CS07103, Library:Tranny_OSC, symbol Tranny_OSC:NX2016SA-52MHZ-EXS00A-CS07103
- C1, C8: footprint Library:01uF_CAP -> Capacitor_SMD:C_0603_1608Metric
- C10: footprint Library:2.2uF_CAP_0603 -> Capacitor_SMD:C_0603_1608Metric
- C11, C12, C13, C14: footprint Library:01uF_Cap_0603 -> Capacitor_SMD:C_0603_1608Metric
- C15, C16, C17, C19, C20, C21, C22: footprint (none) -> Capacitor_SMD:C_0603_1608Metric
- C18, C23, C25: value 100nF -> 0.1uF; footprint (none) -> Capacitor_SMD:C_0603_1608Metric
- C2, C3: footprint Library:0.22Cap -> Capacitor_SMD:C_0603_1608Metric
- C26: footprint (none) -> Capacitor_SMD:C_1206_3216Metric
- C4: footprint Library:22Uf_CAP -> Capacitor_SMD:C_0805_2012Metric
- C5: footprint Library:22Uf_CAP -> Capacitor_SMD:C_0805_2012Metric; now left out of the parts list
- C6, C7: footprint Library:10uF_cap -> Capacitor_SMD:C_1206_3216Metric
- C9: footprint Library:10uF_cap -> Capacitor_SMD:C_0805_2012Metric
- L1: footprint Library:3_3_Inductor -> Library:3.3uH_3.94A
- L2: footprint (none) -> Library:10nH_Inductor
- R1, R2: footprint Library:10kResistor -> Resistor_SMD:R_0603_1608Metric
- R3: footprint Library:33.2Resistor -> Resistor_SMD:R_0603_1608Metric
- R4, R5, R6, R7, R8, R9: footprint (none) -> Resistor_SMD:R_0603_1608Metric
- U1: footprint HTSOP-J8_ROM -> Library:3.3V-LDO (2)
- U11: footprint LIS2MDLTR:PQFN50P200X200X70-12N -> Library:Magnetometer
- U5: footprint DCK0005A_N -> Library:TPS22944 (2)
Connections:
- net GND: now also C36.2, C37.2, C38.1, C39.1, C40.1, J5.N (NEG), M1.3 (-), M2.3 (-), R11.1, U12.1 (GND)
- net GND1: now also C24.2, C27.1, C28.2, C29.2, C30.2, C33.1, C34.2, C35.2, U10.13 (GND__1), U10.20 (GND__2), U10.21 (GND__3), U10.23 (GND__4), U10.24 (GND__5), U10.25 (EXP), U10.5 (GND), XTAL1.2 (GND), XTAL1.3 (GND)
- net SPI_4_SCK: now reaches U4.1 (PE2)
- net SPI_4_SCK: now also U11.1 (SCL/SPC), U3.4 (SCK)
- net SPI_4_CS_MAG: now reaches U4.2 (PE3)
- net SPI_4_CS_MAG: now also U11.3 (CS)
- net SPI_4_NSS_Baro: now reaches U4.3 (PE4)
- net SPI_4_NSS_Baro: now also U3.2 (CSB)
- net RF_Transciever_RESET: now reaches U4.36 (PB2)
- net RF_Transciever_RESET: now also U10.3 (~{RESET})
- net SPI_4_MISO: now reaches U4.4 (PE5)
- net SPI_4_MISO: now also U11.4 (SDA/SDI/SDO), U3.3 (SDI)
- net SPI_4_MOSI: now reaches U4.5 (PE6)
- net SPI_4_MOSI: now also U11.7 (INT/DRDY/SDO), U3.5 (SDO)
- net TIM3_CH1_PWM: now reaches U4.63 (PC6)
- net TIM3_CH1_PWM: now also M1.1 (PWM)
- net TIM3_CH2_PWM: now reaches U4.64 (PC7)
- net TIM3_CH2_PWM: now also M2.1 (PWM)
- net DIO1_EXTI: now reaches U4.83 (PD2)
- net DIO1_EXTI: now also U10.8 (DIO1)
- net DIO2_EXTI: now reaches U4.84 (PD3)
- net DIO2_EXTI: now also U10.9 (DIO2)
- net DIO3_EXTI: now reaches U4.85 (PD4)
- net DIO3_EXTI: now also U10.10 (DIO3)
- net BUSY: now reaches U4.86 (PD5)
- net BUSY: now also U10.7 (BUSY)
- net +9V renamed +15V
- net +15V: now also C38.2, C39.2, C40.2, J5.P (POS), R12.2, U12.3 (VIN)
- net SPI_1_CS_MAG: no longer names the net of U4.34 (PB0)
- net SPI_1_CS_MAG: no longer U11.3 (CS)
- removed net SPI_1_MISO: U11.4 (SDA/SDI/SDO), U3.3 (SDI), U4.90 (PB4(NJTRST))
- removed net SPI_1_MOSI: U11.7 (INT/DRDY/SDO), U3.5 (SDO), U4.91 (PB5)
- net SPI_1_NSS_IMU renamed SPI_1_NSS_Transciever
- net SPI_1_NSS_Transciever: now also U10.19 (~{SS_CTS}); no longer U3.2 (CSB)
- removed net SPI_1_SCK: U11.1 (SCL/SPC), U3.4 (SCK), U4.89 (PB3(JTDO)
- net SPI_2_MISO renamed SPI_2_MISO_IMU
- net SPI_2_MOSI renamed SPI_2_MOSI_IMU
- net SPI_2_NSS renamed SPI_2_NSS_IMU
- net SPI_2_SCK renamed SPI_2_SCK_IMU
- new net: U10.6 (XTB), XTAL1.1
- new net: U10.4 (XTA), XTAL1.3 (GND)
- new net: C41.1, L6.2, U12.2 (SW)
- new net: C41.2, U12.6 (VBST)
- new net: C42.1, R11.2, R13.2, U12.4 (VFB)
- new net: L5.1, U10.14 (DCC_SW)
- new net: C34.1, C35.1, L5.2, U10.12 (DCC_FB), U10.2 (VDD_IN)
- new net: R12.1, U12.5 (EN)
- new net: C24.1, U10.1 (VR_PA)
- new net: C27.2, R10.2, U10.11 (VBAT_IO)
- new net: C28.1, L3.1, U10.22 (RFIO)
- new net: C30.1, C31.2, C32.1, L4.2
- new net: C32.2, J4.1
- new net: C29.1, C31.1, L3.2, L4.1
- new net +6V_Batt: C36.1, C37.1, C42.2, L6.1, M1.2 (+), M2.2 (+), R13.1
- new net 3.3V_Radio: C33.2, R10.1, U10.15 (VBAT)
- new net SPI_1_MISO_Transciever: U10.17 (MOSI_RX), U4.90 (PB4(NJTRST))
- new net SPI_1_MOSI_Transciever: U10.16 (MISO_TX), U4.91 (PB5)
- new net SPI_1_SCK_Transciever: U10.18 (SCK_~{RTS}), U4.89 (PB3(JTDO)
Other:
- note added: "1.0"
- note added: "6V Buck Converter"
- note added: "Flight Controller & Computer"
- note added: "Need to figure out if the SWD 3.3V will power the board as well or if i need a separate power supply. Do I need ESD protection?"
- note added: "Need to route D+/D- w/ ESD diodes and 22 ohm resistors USB C requires 90 0hm impedance paths < 20mm length"
- note added: "RF TRANNY"
- note added: "Servos"
- note added: "XT60-M"
- note added: "djsun"
- note removed: "Need to figure out if the SWD 3.3V will power the board as well or if i need a separate power supply."
- note removed: "Need to route D+/D- w/ ESD diodesand 22 ohm resistors USB C requires 90 0hm impedance paths < 20mm length"
- moved on the sheet: C1, C4, C5, C6, C7, C8, C9, D1, D2, J3, L1, R1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
